File: Hardware/EncoderBoard.kicad_pcb (KiCad board)
At the start: 2 copper layers, 221 x 61 mm, 228 parts, among them SW1 Rotary_Encoder_Switch, SW10 SW_Push_LED_Red, SW11 SW_Push_LED_Blue, SW12 SW_Push_LED_Red, SW13 SW_Push_LED_Yellow, SW14 SW_Push_LED_Green, SW15 SW_Push_LED_Blue, SW2 Rotary_Encoder_Switch, SW3 Rotary_Encoder_Switch, SW4 Rotary_Encoder_Switch, SW5 Rotary_Encoder_Switch, SW6 Rotary_Encoder_Switch, SW7 Rotary_Encoder_Switch, SW8 Rotary_Encoder_Switch, SW9 Rotary_Encoder_Switch, U1 MCP23S17_SO, U10 Display_OLED_128x32_I2C, U11 Display_OLED_128x32_I2C, U12 Display_OLED_128x32_I2C, U13 Display_OLED_128x32_I2C, U14 Display_OLED_128x32_I2C, U15 Display_OLED_128x32_I2C, U16 Display_OLED_128x32_I2C, U17 Display_OLED_128x32_I2C, U18 74LVC14, U19 74LVC14, U2 MCP23S17_SO, U20 74LVC14, U21 74LVC14, U22 74LVC14, U23 74LVC14, U24 CAT24M01W, U25 CAT24M01W, U26 CAT24M01W, U3 MCP23S17_SO, U4 TCA9548APWR, U5 74HCT245, U6 TCA9548APWR, U7 Teensy3.2, U8 CAT24M01W, U9 Display_OLED_128x32_I2C

Commit message: Progress push Rev C PCB
Change Buttons to Gateron/Cherry MX and WS2812 as part of key
Teensy 4.0 Compatible design / Under mount Teensy
Update Read Me with work in progress list
Add symbols to PCB with common values for easier soldering
Parts:
- removed R26, R38: 150, Resistor_BG:R_0805_2012Metric
- removed R31, R51: 33, Resistor_BG:R_0805_2012Metric
- removed R41, R48: 120, Resistor_BG:R_0805_2012Metric
- removed REF** (x5): MountingHole_3.2mm_M3, MountingHole:MountingHole_3.2mm_M3
- removed SW10: SW_Push_LED_Red, Button_Switch_BG:E-Switch_SPST_Red_LED_RoundCap_TL3240F160R
- removed SW11: SW_Push_LED_Blue, Button_Switch_BG:E-Switch_SPST_LED_RoundCap_TL3240F160x
- removed SW12: SW_Push_LED_Red, Button_Switch_BG:E-Switch_SPST_Red_LED_SquareCap_TL3240F160R
- removed SW13: SW_Push_LED_Yellow, Button_Switch_BG:E-Switch_SPST_LED_SquareCap_TL3240F160x
- removed SW14: SW_Push_LED_Green, Button_Switch_BG:E-Switch_SPST_LED_SquareCap_TL3240F160x
- removed SW15: SW_Push_LED_Blue, Button_Switch_BG:E-Switch_SPST_LED_SquareCap_TL3240F160x
- added C76: 0.1uf, Capacitor_SMD:C_0805_2012Metric_Pad1.18x1.45mm_HandSolder, F.Cu at (244.8, 69.7)
- added C77: C, Capacitor_SMD:C_0805_2012Metric_Pad1.18x1.45mm_HandSolder, F.Cu at (264.0, 69.7)
- added C78: 0.1uf, Capacitor_SMD:C_0805_2012Metric_Pad1.18x1.45mm_HandSolder, F.Cu at (244.8, 88.8)
- added C79: 0.1uf, Capacitor_SMD:C_0805_2012Metric_Pad1.18x1.45mm_HandSolder, F.Cu at (263.9, 88.8)
- added C80: 0.1uf, Capacitor_SMD:C_0805_2012Metric_Pad1.18x1.45mm_HandSolder, F.Cu at (244.8, 107.8)
- added C81: 0.1uf, Capacitor_SMD:C_0805_2012Metric_Pad1.18x1.45mm_HandSolder, F.Cu at (263.9, 107.8)
- added H1: MountingHole, MountingHole:MountingHole_3.2mm_M3, F.Cu at (33.5, 103.9)
- added H2: MountingHole, MountingHole:MountingHole_3.2mm_M3, F.Cu at (65.5, 56.9)
- added H3: MountingHole, MountingHole:MountingHole_3.2mm_M3, F.Cu at (105.5, 56.9)
- added H4: MountingHole, MountingHole:MountingHole_3.2mm_M3, F.Cu at (181.5, 56.9)
- added H5: MountingHole, MountingHole:MountingHole_3.2mm_M3, F.Cu at (229.5, 92.9)
- added K1: key, kicad custom footprints:SW_Cherry_MX_1.00u_Plate, F.Cu at (247.4, 56.1)
- added K2: key, kicad custom footprints:SW_Cherry_MX_1.00u_Plate, F.Cu at (266.5, 56.1)
- added K3: key, kicad custom footprints:SW_Cherry_MX_1.00u_Plate, F.Cu at (247.4, 75.2)
- added K4: key, kicad custom footprints:SW_Cherry_MX_1.00u_Plate, F.Cu at (266.4, 75.2)
- added K5: key, kicad custom footprints:SW_Cherry_MX_1.00u_Plate, F.Cu at (247.4, 94.2)
- added K6: key, kicad custom footprints:SW_Cherry_MX_1.00u_Plate, F.Cu at (266.4, 94.2)
- C18, C25, C28, C45, C52, C54, R36, R53, R64, R67, R80, R86, R90, R91, R92, R93, R94, R95, U7: moved to B.Cu
- moved C54 199.9 mm to (258.0, 100.0), turned to 90 degrees
- moved R86 194.2 mm to (255.8, 100.0), turned to 90 degrees
- moved R95 193.3 mm to (255.8, 96.2)
- moved R93 192.9 mm to (255.8, 77.2)
- moved C45 192.7 mm to (258.0, 81.0), turned to 90 degrees
- moved R92 191.3 mm to (253.0, 77.2)
- moved C28 190.9 mm to (250.8, 80.9), turned to 90 degrees
- moved R94 190.6 mm to (253.0, 96.2)
- moved R67 190.4 mm to (255.8, 81.0), turned to 90 degrees
- moved R64 189.3 mm to (253.0, 80.9)
- moved R80 188.7 mm to (253.0, 100.0)
- moved C52 186.3 mm to (250.8, 100.0), turned to 90 degrees
- moved C61 35.5 mm to (205.5, 81.5), turned to 90 degrees
- moved C6 34.5 mm to (232.1, 86.4)
- moved C5 34.5 mm to (227.9, 87.7)
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Connections:
- D1 pad 2: Net-(D1-Pad2) -> (no net)
- D10 pad 2: Net-(D10-Pad2) -> (no net)
- D10 pad 4: Net-(D10-Pad4) -> (no net)
- D11 pad 2: Net-(D11-Pad2) -> (no net)
- D11 pad 4: Net-(D10-Pad2) -> (no net)
- D12 pad 2: (no net) -> KEY_WS_DATA
- D12 pad 4: Net-(D11-Pad2) -> (no net)
- D2 pad 2: Net-(D2-Pad2) -> (no net)
- D2 pad 4: Net-(D1-Pad2) -> (no net)
- D3 pad 2: Net-(D3-Pad2) -> (no net)
- D3 pad 4: Net-(D2-Pad2) -> (no net)
- D4 pad 2: Net-(D4-Pad2) -> (no net)
- D4 pad 4: Net-(D3-Pad2) -> (no net)
- D5 pad 2: Net-(D5-Pad2) -> (no net)
- D5 pad 4: Net-(D4-Pad2) -> (no net)
- D6 pad 2: Net-(D6-Pad2) -> (no net)
- D6 pad 4: Net-(D5-Pad2) -> (no net)
- D7 pad 2: Net-(D7-Pad2) -> (no net)
- D7 pad 4: Net-(D6-Pad2) -> (no net)
- D8 pad 2: Net-(D8-Pad2) -> (no net)
- D8 pad 4: Net-(D7-Pad2) -> (no net)
- D9 pad 2: Net-(D10-Pad4) -> (no net)
- D9 pad 4: Net-(D8-Pad2) -> (no net)
- U1 pad 19: (no net) -> unconnected-(U1-INTB-Pad19)
- U1 pad 24: (no net) -> unconnected-(U1-GPA3-Pad24)
- U1 pad 28: (no net) -> unconnected-(U1-GPA7-Pad28)
- U1 pad 4: (no net) -> unconnected-(U1-GPB3-Pad4)
- U1 pad 8: (no net) -> unconnected-(U1-GPB7-Pad8)
- U2 pad 19: (no net) -> unconnected-(U2-INTB-Pad19)
- U2 pad 24: (no net) -> unconnected-(U2-GPA3-Pad24)
- U2 pad 28: (no net) -> unconnected-(U2-GPA7-Pad28)
- U2 pad 4: (no net) -> unconnected-(U2-GPB3-Pad4)
- U2 pad 8: (no net) -> unconnected-(U2-GPB7-Pad8)
- U24 pad 1: (no net) -> unconnected-(U24-NC-Pad1)
- U25 pad 1: (no net) -> unconnected-(U25-NC-Pad1)
- U26 pad 1: (no net) -> unconnected-(U26-NC-Pad1)
- U3 pad 1: (no net) -> unconnected-(U3-GPB0-Pad1)
- U3 pad 19: (no net) -> unconnected-(U3-INTB-Pad19)
- U3 pad 2: (no net) -> unconnected-(U3-GPB1-Pad2)
- U3 pad 28: (no net) -> unconnected-(U3-GPA7-Pad28)
- U3 pad 3: (no net) -> unconnected-(U3-GPB2-Pad3)
- U3 pad 4: (no net) -> unconnected-(U3-GPB3-Pad4)
- U3 pad 5: (no net) -> unconnected-(U3-GPB4-Pad5)
- U3 pad 6: (no net) -> unconnected-(U3-GPB5-Pad6)
- U4 pad 10: (no net) -> unconnected-(U4-SD3-Pad10)
- U4 pad 11: (no net) -> unconnected-(U4-SC3-Pad11)
- U4 pad 19: (no net) -> unconnected-(U4-SD7-Pad19)
- U4 pad 20: (no net) -> unconnected-(U4-SC7-Pad20)
- U5 pad 11: (no net) -> unconnected-(U5-B7-Pad11)
- U5 pad 12: (no net) -> unconnected-(U5-B6-Pad12)
- U5 pad 13: (no net) -> unconnected-(U5-B5-Pad13)
- U5 pad 14: (no net) -> unconnected-(U5-B4-Pad14)
- U5 pad 15: (no net) -> unconnected-(U5-B3-Pad15)
- U5 pad 16: (no net) -> unconnected-(U5-B2-Pad16)
- U5 pad 17: (no net) -> unconnected-(U5-B1-Pad17)
- U5 pad 3: (no net) -> unconnected-(U5-A1-Pad3)
- U5 pad 4: (no net) -> unconnected-(U5-A2-Pad4)
- U5 pad 5: (no net) -> unconnected-(U5-A3-Pad5)
- U5 pad 6: (no net) -> unconnected-(U5-A4-Pad6)
- U5 pad 7: (no net) -> unconnected-(U5-A5-Pad7)
- U5 pad 8: (no net) -> unconnected-(U5-A6-Pad8)
- U5 pad 9: (no net) -> unconnected-(U5-A7-Pad9)
- U6 pad 10: (no net) -> unconnected-(U6-SD3-Pad10)
- U6 pad 11: (no net) -> unconnected-(U6-SC3-Pad11)
- U6 pad 15: (no net) -> unconnected-(U6-SD5-Pad15)
- U6 pad 16: (no net) -> unconnected-(U6-SC5-Pad16)
- U6 pad 17: (no net) -> unconnected-(U6-SD6-Pad17)
- U6 pad 18: (no net) -> unconnected-(U6-SC6-Pad18)
- U6 pad 19: (no net) -> unconnected-(U6-SD7-Pad19)
- U6 pad 20: (no net) -> unconnected-(U6-SC7-Pad20)
- U6 pad 8: (no net) -> unconnected-(U6-SD2-Pad8)
- U6 pad 9: (no net) -> unconnected-(U6-SC2-Pad9)
- U7 pad 15: (no net) -> unconnected-(U7-VBat-Pad15)
- U7 pad 16: (no net) -> unconnected-(U7-3.3V-Pad16)
- U7 pad 18: (no net) -> unconnected-(U7-Program-Pad18)
- U7 pad 19: (no net) -> unconnected-(U7-A14/DAC-Pad19)
- U7 pad 2: (no net) -> unconnected-(U7-0_RX1_Touch-Pad2)
- U7 pad 21: (no net) -> unconnected-(U7-14_A0_SCK-Pad21)
- U7 pad 22: (no net) -> unconnected-(U7-15_A1_CS_Touch-Pad22)
- U7 pad 23: (no net) -> unconnected-(U7-16_A2_SCL0_Touch-Pad23)
- U7 pad 24: (no net) -> unconnected-(U7-17_A3_SDA0_Touch-Pad24)
- U7 pad 27: BUTTON2_LED -> unconnected-(U7-20_A6_CS_PWM-Pad27)
- U7 pad 28: BUTTON3_LED -> unconnected-(U7-21_A7_RX1_CS_PWM-Pad28)
- U7 pad 29: BUTTON4_LED -> unconnected-(U7-22_A8_Touch_PWM-Pad29)
- U7 pad 30: BUTTON5_LED -> unconnected-(U7-23_A9_Touch_PWM-Pad30)
- U7 pad 5: (no net) -> unconnected-(U7-3_TX_PWM-Pad5)
- U7 pad 6: (no net) -> unconnected-(U7-4_RX_PWM-Pad6)
- U7 pad 7: BUTTON0_LED -> unconnected-(U7-5_TX1_PWM-Pad7)
- U7 pad 8: BUTTON1_LED -> unconnected-(U7-6_PWM-Pad8)
- U8 pad 1: (no net) -> unconnected-(U8-NC-Pad1)
Routing:
- net GND: track 711.8 -> 103.0 mm, vias 38 -> 39
- net (no net): track 0.00 -> 368.0 mm, vias 5 -> 4
- net BUTTON5_LED: track 267.6 -> 0.00 mm
- net BUTTON4_LED: track 249.4 -> 0.00 mm
- net BUTTON3_LED: track 231.9 -> 0.00 mm
- net BUTTON2_LED: track 223.0 -> 0.00 mm
- net +3V3: track 1074.6 -> 1277.3 mm, vias 24 -> 19
- net Net-(C45-Pad1): track 248.6 -> 46.6 mm, vias 1 -> 0
- net Net-(C28-Pad1): track 243.4 -> 41.9 mm, vias 1 -> 0
- net Net-(C52-Pad1): track 209.1 -> 42.1 mm, vias 1 -> 0
- net Net-(C54-Pad1): track 197.6 -> 58.4 mm, vias 1 -> 0
- net +5V: track 567.3 -> 701.8 mm
- net KEY_WS_DATA: track 0.00 -> 94.1 mm
- net Net-(C18-Pad1): track 31.5 -> 95.0 mm, vias 1 -> 2
- net Net-(D8-Pad2): track 61.3 -> 0.00 mm
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- added copper zone on F.Cu, net GND
Other:
- board size 221 x 61 mm -> 243.8 x 61 mm
- net class Default removed
- net class Power_3V3 removed
- net class Power_5V removed
- board text added: "100nf"
- board text added: "10k"
- board text added: "10nf"
- board text added: "10uf"
- board text added: "4.7k"
- board text added: "Encoder Board Blake Garner & Geoff Evans Rev C Jun 2024"
- board text removed: "Encoder Board Blake Garner Rev B 2 Jun 2020"
